File: board/Pico_TOSLINK_IR.kicad_sch (KiCad schematic)
At the start: 32 parts, among them J4 JTAG_TC2030, J5 BM02B-ACHSS-GAN-TF, U10 W25Q128JVS, U2 apple tv tos link, U7 IRM-V838M3-C/TR1, U8 RP2040, Y1 12MHz

Commit message: worked on new version with rp2350
Parts:
- removed C18, C8: 100n, Capacitor_SMD:C_0402_1005Metric, symbol Device:C_Small
- removed U10: W25Q128JVS, Package_SO:SOIC-8_5.23x5.23mm_P1.27mm, symbol Memory_Flash:W25Q128JVS
- removed U8: RP2040, Package_DFN_QFN:QFN-56-1EP_7x7mm_P0.4mm_EP3.2x3.2mm, symbol Sleep-lib:RP2040
- added C10, C11, C8: 4.7u, Capacitor_SMD:C_0402_1005Metric, symbol Device:C
- added L2: 3.3u, Inductor_SMD:L_Murata_DFE201610P, symbol Device:L
- added R12: 33, Resistor_SMD:R_0402_1005Metric, symbol Device:R
- added R13: 10K, Resistor_SMD:R_0402_1005Metric, symbol Device:R
- added U4: RP2350A-QFN60, Package_DFN_QFN:QFN-60-1EP_7x7mm_P0.4mm_EP3.4x3.4mm, symbol rp2350:RP2350A-QFN60
- C19: value 1u -> 4.7u
- C21: value 10u -> 100n
- C22: value 1u -> 100n
- C29, C30: value 22pF -> 15pF
- Y1: value 12MHz -> ABM8-272-T3
Connections:
- net +1V1: now also C20.1, C11.1, L2.1, U4.23 (DVDD), U4.39 (DVDD), U4.50 (VREG_FB), U4.6 (DVDD)
- net +3V3: now also C10.1, R12.1, R13.1, U4.1 (IOVDD), U4.11 (IOVDD), U4.20 (IOVDD), U4.30 (IOVDD), U4.38 (IOVDD), U4.44 (ADC_AVDD), U4.45 (IOVDD), U4.49 (VREG_VIN), U4.53 (USB_OTP_VDD), U4.54 (QSPI_IOVDD); no longer C20.1
- net GND: now also C10.2, C11.2, C8.2, U4.47 (VREG_PGND), U4.61 (GND)
- net PICO_LED: now also U4.37 (GPIO25)
- net Pico_rx: now also U4.3 (GPIO1)
- net Pico_scl: now also U4.10 (GPIO7)
- net Pico_sda: now also U4.9 (GPIO6)
- net Pico_tx: now also U4.2 (GPIO0)
- net SWCLK: now also U4.24 (SWCLK)
- net SWD: now also U4.25 (SWDIO)
- net XTAL_IN: now also U4.21 (XIN)
- net XTAL_OUT: now also U4.22 (XOUT)
- net toslink: now also U4.16 (GPIO12)
- net ~{RESET}: now also U4.26 (RUN)
- net at R3.2, U7.3 (OUT): now also U4.42 (GPIO28_ADC2)
- net at R8.1: now also U4.31 (GPIO19)
- new net: L2.2, U4.48 (VREG_LX)
- new net: C8.1, R12.2, U4.46 (VREG_AVDD)
- new net: R13.2, U4.60 (QSPI_SS)
- no-connect marks 19 -> 39
Other:
- note added: "RP2354A Chip"
- note removed: "Flash Memory"
- note removed: "RP2040 Chip"
- moved on the sheet: C17, C19, C21, C22, C23, C24, C25, C26, C27, C29, C30, C5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

Commit message: updated most stuff, but i completely redid the diff pairs
Connections:
- net +3V3: no longer J4.1 (VCC)
- no-connect marks 39 -> 41
Changed lines of the file:
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@@
 	)
 	(no_connect
+		(at 36.83 179.07)
+	)
+	(no_connect
 		(at 156.21 132.08)
 	)
@@
 	)
 	(no_connect
+		(at 48.26 166.37)
+	)
+	(no_connect
 		(at 275.59 80.01)
 	)
@@
 	(wire
 		(pts
-			(xy 48.26 163.83) (xy 48.26 166.37)
-		)
-		(stroke
-			(width 0)
-			(type default)
-		)
-	)
-	(wire
-		(pts
 			(xy 189.23 38.1) (xy 195.58 38.1)
 		)
@@
 					(unit 1)
 				)
-			)
-		)
-	)
-	(symbol
-		(lib_id "power:+3V3")
-		(at 48.26 163.83 0)
-		(unit 1)
-		(exclude_from_sim no)
-		(in_bom yes)
-		(on_board yes)
-		(dnp no)
-		(property "Reference" "#PWR046"
-			(at 48.26 167.64 0)
-			(effects
-				(font
-					(size 1.27 1.27)
-				)
-				(hide yes)
-			)
-		)
-		(property "Value" "+3V3"
-			(at 48.26 160.528 0)
-			(effects
-				(font
-					(size 1.27 1.27)
-				)
-			)
-		)
-		(property "Footprint" ""
-			(at 48.26 163.83 0)
-			(effects
-				(font
-					(size 1.27 1.27)
-				)
-				(hide yes)
-			)
-		)
-		(property "Datasheet" ""
-			(at 48.26 163.83 0)
-			(effects
-				(font
-					(size 1.27 1.27)
-				)
-				(hide yes)
-			)
-		)
-		(property "Description" "Power symbol creates a global label with name \"+3V3\""
-			(at 48.26 163.83 0)
-			(effects
-				(font
-					(size 1.27 1.27)
-				)
-				(hide yes)
-			)
-		)
-		(pin "1"
-		)
-		(instances
-			(project "apple_pi_tv_board"
-				(path "/391fcf0b-b604-4ad0-921e-8f3dad9a49eb/ffa30f6a-e405-44ad-a0eb-1eb85feaca3b"
-					(reference "#PWR046")
-					(unit 1)
-				)

Commit message: almost v0.3
Parts:
- U4: value RP2350A-QFN60 -> RP2354A
Changed lines of the file:
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@@
 			)
 		)
-		(property "Description" "AOTA-B201610S3R3-101-T"
+		(property "Description" "Abracon AOTA-B201610S3R3-101-T"
 			(at 59.69 58.42 0)
 			(effects
@@
 			)
 		)
-		(property "Value" "RP2350A-QFN60"
+		(property "Value" "RP2354A"
 			(at 127.8733 148.59 0)
 			(effects
