File: board/Pico_TOSLINK_IR.kicad_sch (KiCad schematic)
At the start: 35 parts, among them J4 JTAG_TC2030, J5 BM02B-ACHSS-GAN-TF, U2 apple tv tos link, U4 RP2354A, U7 IRM-V838M3-C/TR1, Y1 ABM8-272-T3

Commit message: most schematic is done
Parts:
- removed J4: JTAG_TC2030, Connector:Tag-Connect_TC2030-IDC-NL_2x03_P1.27mm_Vertical, symbol marbastlib-various:JTAG_TC2030
- added J2: Dev_port, Connector:Tag-Connect_TC2030-IDC-NL_2x03_P1.27mm_Vertical, symbol apple_tv_parts:dev_connector
- added R18, R19: 220R, Resistor_SMD:R_0402_1005Metric, symbol Device:R_Small_US
- J5: value BM02B-ACHSS-GAN-TF -> HDGC1202WR-S-2P; footprint greencharge-footprints:BM02BSRSSTBLFSN -> HDGC:HDGC1202WR-S-02P
- R7: value 470R -> 10K R
- U2: now not fitted
Connections:
- net +3V3: now also R18.1, R19.1
- net GND: now also J5.mp, J2.6 (GND)
- net Pico_scl: now also U4.33 (GPIO21); no longer U4.10 (GPIO7)
- net Pico_sda: now also U4.32 (GPIO20); no longer U4.9 (GPIO6)
- net Pico_tx: now also J2.4 (Pico_Tx)
- net SWCLK: now also J2.2 (SWCLK)
- net SWD: now also J2.1 (SWD)
- net ~{RESET}: now also J2.3 (RST)
- net I2S_clk: now reaches U4.12 (GPIO8)
- net I2S_LRCLK: now reaches U4.13 (GPIO9)
- net I2S_DOUT: now reaches U4.14 (GPIO10)
- net pico_hid_irq: now reaches U4.15 (GPIO11)
- net Pico_blinky: now reaches R8.1, U4.31 (GPIO19)
- new net PI_eeprom_scl: R19.2, U4.10 (GPIO7)
- new net PI_eeprom_sda: R18.2, U4.9 (GPIO6)
- new net Pi_tx: J2.5 (Pi_Tx)
- no-connect marks 41 -> 33
Other:
- note added: "Case LED"
- note removed: "LED"

Commit message: almost ready to send out
Connections:
- net GND: now also J2.1 (GND), J5.MP; no longer J2.6 (GND), J5.mp
- net Pi_tx: now also J2.3 (Pi_Tx); no longer J2.5 (Pi_Tx)
- net Pico_tx: now also J2.5 (Pico_Tx); no longer J2.4 (Pico_Tx)
- net SWCLK: now also J2.4 (SWCLK); no longer J2.2 (SWCLK)
- net SWD: now also J2.2 (SWD); no longer J2.1 (SWD)
- net ~{RESET}: now also J2.6 (RST); no longer J2.3 (RST)
Changed lines of the file:
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@@
 		(pin "2"
 		)
-		(pin "mp"
+		(pin "MP"
 		)
 		(instances
