File: board/HDMI_RJ45_USB.kicad_sch (KiCad schematic)
At the start: 19 parts, among them J1 RJ45_Shielded, T1 H5007NL, U1 HDMI/USB, U11 TPD4EUSB30, U12 RT9742GGJ5, U5 RT9742GGJ5, U6 TPD4EUSB30

Commit message: most schematic is done
Parts:
- J1, U1: now not fitted
Changed lines of the file:
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@@
 		(in_bom yes)
 		(on_board yes)
-		(dnp no)
+		(dnp yes)
 		(property "Reference" "J1"
 			(at 259.334 40.894 0)
@@
 		(in_bom no)
 		(on_board yes)
-		(dnp no)
+		(dnp yes)
 		(property "Reference" "U1"
 			(at 86.614 44.704 0)
