File: board/Power.kicad_sch (KiCad schematic)
At the start: 9 parts, among them J3 5-1775444-8, U9 TPS61232DRC

Commit message: most schematic is done
Parts:
- added C18: 4.7u, Capacitor_SMD:C_0402_1005Metric, symbol Device:C_Small
- added C32, C33: 22u, Capacitor_SMD:C_0402_1005Metric, symbol Device:C_Small
- C12: value 8.2n -> 8.2nf
Connections:
- net +5V: now also C18.1, C32.1, C33.1
- net GND: now also C18.2, C32.2, C33.2
