File: board/apple_pi_tv_board.kicad_pcb (KiCad board)
At the start: 4 copper layers, 61 x 85.1 mm, 78 parts, among them J1 RJ45_Shielded, J3 5-1775444-8, J4 JTAG_TC2030, J5 BM02B-ACHSS-GAN-TF, T1 H5007NL, U1 HDMI/USB, U11 TPD4EUSB30, U12 RT9742GGJ5, U2 apple tv tos link, U3 RPi_4, U4 RP2354A, U5 RT9742GGJ5, U6 TPD4EUSB30, U7 IRM-V838M3-C/TR1, U8 74LVC1G07, U9 TPS61232DRC, Y1 ABM8-272-T3

Commit message: most schematic is done
Parts:
- removed J4: JTAG_TC2030, Connector:Tag-Connect_TC2030-IDC-NL_2x03_P1.27mm_Vertical
- removed JP3-EEPROM1: SolderJumper_2_Open, Jumper:SolderJumper-2_P1.3mm_Open_TrianglePad1.0x1.5mm
- added C18: 4.7u, Capacitor_SMD:C_0402_1005Metric, F.Cu at (110.8, 141.7)
- added C32: 22u, Capacitor_SMD:C_0402_1005Metric, F.Cu at (109.8, 141.7)
- added C33: 22u, Capacitor_SMD:C_0402_1005Metric, F.Cu at (108.8, 141.7)
- added J2: Dev_port, Connector:Tag-Connect_TC2030-IDC-NL_2x03_P1.27mm_Vertical, F.Cu at (135.0, 147.6)
- added R18: 220R, Resistor_SMD:R_0402_1005Metric, F.Cu at (107.8, 126.1)
- added R19: 220R, Resistor_SMD:R_0402_1005Metric, F.Cu at (109.7, 126.0)
- C12: value 8.2n -> 8.2nf
- H1: footprint MountingHole:MountingHole_2.7mm_Pad -> apple_tv_parts:ExtendedMountingHole
- J5: value BM02B-ACHSS-GAN-TF -> HDGC1202WR-S-2P; footprint greencharge-footprints:BM02BSRSSTBLFSN -> HDGC:HDGC1202WR-S-02P
- R7: value 470R -> 10K R
- moved R2 5.81 mm to (129.0, 134.5)
- moved R3 5.81 mm to (131.0, 134.5)
- moved C5 4.31 mm to (127.0, 136.0)
- moved U8 1.98 mm to (135.8, 95.3)
- moved U7 1.79 mm to (128.9, 140.4)
- moved R9 1.76 mm to (138.4, 95.9)
- moved J5 1.59 mm to (123.8, 146.6)
- moved D2 1.41 mm to (137.1, 92.0), turned to 180 degrees
- moved U12 1.28 mm to (137.2, 80.7)
- moved R6 1.22 mm to (137.3, 83.4)
- moved H1 0.96 mm to (135.4, 87.9)
- moved C4 0.41 mm to (85.0, 114.2)
Connections:
- net Net-(U4-GPIO19) renamed /Pico_TOSLINK_IR/Pico_blinky
- U3 pad 20: Net-(JP3-EEPROM1-B) -> GND
- U3 pad 25: /HDMI_PWR_ON -> /I2S_OUT
- U3 pad 26: unconnected-(U3A-GPIO19-Pad26) -> /I2S_LRCLK
- U3 pad 28: unconnected-(U3A-GPIO13-Pad28) -> /Pico_scl
- U3 pad 30: unconnected-(U3A-GPIO6-Pad30) -> /Pico_hid_irq
- U3 pad 35: unconnected-(U3A-ID_SC-Pad35) -> /PI_eeprom_scl
- U3 pad 36: unconnected-(U3A-ID_SD-Pad36) -> /Pi_eeprom_sda
- U3 pad 38: unconnected-(U3A-GPIO11-Pad38) -> /Pico_sda
- U3 pad 49: unconnected-(U3A-GPIO18-Pad49) -> /I2S_CLK
- U3 pad 51: /pico_tx -> /PI_UART_TX
- U3 pad 54: unconnected-(U3A-GPIO4-Pad54) -> /pico_rx
- U3 pad 55: /pico_rx -> /PI_UART_RX
- U3 pad 64: unconnected-(U3A-SD_DAT5-Pad64) -> /pico_tx
- U3 pad 80: /Pico_scl -> unconnected-(U3A-SCL0-Pad80)
- U3 pad 82: /Pico_sda -> unconnected-(U3A-SDA0-Pad82)
- U4 pad 10: /Pico_scl -> /PI_eeprom_scl
- U4 pad 12: unconnected-(U4-GPIO8-Pad12) -> /I2S_CLK
- U4 pad 13: unconnected-(U4-GPIO9-Pad13) -> /I2S_LRCLK
- U4 pad 14: unconnected-(U4-GPIO10-Pad14) -> /I2S_OUT
- U4 pad 15: unconnected-(U4-GPIO11-Pad15) -> /Pico_hid_irq
- U4 pad 32: unconnected-(U4-GPIO20-Pad32) -> /Pico_sda
- U4 pad 33: unconnected-(U4-GPIO21-Pad33) -> /Pico_scl
- U4 pad 9: /Pico_sda -> /Pi_eeprom_sda
Routing:
- net /HDMI_PWR_ON: track 80.9 -> 1.75 mm, vias 2 -> 0
- net /I2S_OUT: track 0.00 -> 19.2 mm, vias 0 -> 2
- net +5V: track 108.2 -> 121.5 mm
- net Net-(JP3-EEPROM1-B): track 12.9 -> 0.00 mm, vias 2 -> 0
- net Net-(U4-GPIO28_ADC2): track 40.2 -> 45.4 mm
- net Net-(U7-VCC): track 2.89 -> 6.96 mm
- net +3V3: track 208.6 -> 212.0 mm
- net /Pico_TOSLINK_IR/~{RESET}: track 64.4 -> 67.5 mm
- net GND: track 162.6 -> 164.9 mm, vias 95 -> 94
- net Net-(D2-K): track 1.69 -> 3.51 mm
- net Net-(U3A-PI_LED_~{PWR}): track 49.8 -> 48.4 mm
- net /SD_DAT2: track 52.2 -> 53.4 mm
- net /SD_PWR_ON: track 33.1 -> 33.8 mm
- net /HDMI_RJ45_USB/HDMI_5v: track 47.1 -> 46.4 mm

Commit message: almost ready to send out
Parts:
- added J4: DF40C-100DS-0.4V_51_, Hirose:HIROSE_DF40C-100DS-0.4V_51_, F.Cu at (110.7, 96.2)
- added J6: DF40C-100DS-0.4V_51_, Hirose:HIROSE_DF40C-100DS-0.4V_51_, F.Cu at (110.7, 130.3)
- moved R19 11.8 mm to (106.1, 137.2), turned to 90 degrees
- moved J2 4.57 mm to (135.6, 143.1), turned to 90 degrees
- moved C26 0.61 mm to (98.2, 137.6), turned to 90 degrees
- moved R18 0.17 mm to (107.7, 126.2)
Connections:
- J2 pad 1: (no net) -> GND
- J2 pad 2: (no net) -> /swdio
- J2 pad 3: (no net) -> /PI_UART_TX
- J2 pad 4: (no net) -> /swclk
- J2 pad 5: (no net) -> /pico_tx
- J2 pad 6: (no net) -> /Pico_TOSLINK_IR/~{RESET}
- J5 pad MP: (no net) -> GND
Routing:
- net /PI_UART_TX: track 0.00 -> 48.5 mm, vias 0 -> 2
- net /pico_tx: track 14.2 -> 59.2 mm, vias 2 -> 3
- net /Pico_hid_irq: track 0.00 -> 21.6 mm, vias 0 -> 3
- net /I2S_CLK: track 0.00 -> 20.3 mm, vias 0 -> 2
- net /Pi_eeprom_sda: track 0.00 -> 19.0 mm, vias 0 -> 2
- net /I2S_LRCLK: track 0.00 -> 17.4 mm, vias 0 -> 2
- net /PI_eeprom_scl: track 0.00 -> 17.2 mm, vias 0 -> 3
- net /Pico_scl: track 28.0 -> 37.0 mm
- net /I2S_OUT: track 19.2 -> 15.0 mm
- net /Pico_TOSLINK_IR/~{RESET}: track 67.5 -> 63.5 mm
- net +3V3: track 212.0 -> 215.8 mm, vias 22 -> 24
- net /pico_rx: track 18.7 -> 22.3 mm
- net /swdio: track 86.9 -> 84.4 mm
- net /Pico_sda: track 28.9 -> 31.3 mm
- net GND: track 164.9 -> 166.1 mm
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Other:
- board text added: "REV .4"
