File: board/apple_pi_tv_board.kicad_sch (KiCad schematic)
At the start: 15 parts, among them U3 RPi_4, U8 74LVC1G07

Commit message: most schematic is done
Parts:
- removed JP3-EEPROM1: SolderJumper_2_Open, Jumper:SolderJumper-2_P1.3mm_Open_TrianglePad1.0x1.5mm, symbol Jumper:SolderJumper_2_Open
- added J4, J6: DF40C-100DS-0.4V_51_, DF40C-100DS-0.4V_51_:HIROSE_DF40C-100DS-0.4V_51_, symbol Hirose:DF40C-100DS-0.4V_51_
- H1: footprint MountingHole:MountingHole_2.7mm_Pad -> apple_tv_parts:ExtendedMountingHole
- U3: now not fitted
Connections:
- net GND: now also U3.20 (EEPROM_~{WP})
- net HDMI_PWR_ON: no longer U3.25 (GPIO21)
- net Pico_scl: now also U3.28 (GPIO13); no longer U3.80 (SCL0)
- net Pico_sda: now also U3.38 (GPIO11); no longer U3.82 (SDA0)
- net pico_rx: now also U3.54 (GPIO4); no longer U3.55 (GPIO14)
- net pico_tx: now also U3.64 (SD_DAT5); no longer U3.51 (GPIO15)
- net I2S_LRCLK: now reaches U3.26 (GPIO19)
- net Pico_hid_irq: now reaches U3.30 (GPIO6)
- net PI_eeprom_scl: now reaches U3.35 (ID_SC)
- net Pi_eeprom_sda: now reaches U3.36 (ID_SD)
- net I2S_CLK: now reaches U3.49 (GPIO18)
- new net I2S_OUT: U3.25 (GPIO21)
- new net PI_UART_RX: U3.55 (GPIO14)
- new net PI_UART_TX: U3.51 (GPIO15)
Other:
- sheet Pico_TOSLINK_IR ports: added I2S_DOUT, I2S_LRCLK, I2S_clk, PI_eeprom_scl, PI_eeprom_sda, Pi_tx, pico_hid_irq; removed none

Commit message: almost ready to send out
Parts:
- J4, J6: footprint DF40C-100DS-0.4V_51_:HIROSE_DF40C-100DS-0.4V_51_ -> Hirose:HIROSE_DF40C-100DS-0.4V_51_
Changed lines of the file:
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@@
 			)
 		)
-		(property "Footprint" "DF40C-100DS-0.4V_51_:HIROSE_DF40C-100DS-0.4V_51_"
+		(property "Footprint" "Hirose:HIROSE_DF40C-100DS-0.4V_51_"
 			(at 185.42 284.48 0)
 			(effects
@@
 			)
 		)
-		(property "Footprint" "DF40C-100DS-0.4V_51_:HIROSE_DF40C-100DS-0.4V_51_"
+		(property "Footprint" "Hirose:HIROSE_DF40C-100DS-0.4V_51_"
 			(at 100.33 280.67 0)
 			(effects
